File: hardware/iq_modulator.sch (KiCad schematic (older format))
At the start: 1 part

Commit message: Update PA matching circuits
Parts:
- added C15: 100pF, symbol device:C
- added C19, C22, C24, C26, C28, C30, C31, C32, C34, C36, C38, C4, C40: 100n, Capacitors_SMD:C_0603, symbol device:C_Small
- added C23, C25, C27, C29, C33, C35, C37, C39, C41, C7: 10p, Capacitors_SMD:C_0603, symbol device:C_Small
- added C42: 220µF, symbol device:CP
- added D2: LED, LEDs:LED_0603, symbol device:LED
- added R5: 4k7, Resistors_SMD:R_0603, symbol device:R
- added R6: 100, Resistors_SMD:R_0603, symbol device:R
- added TP1: MUXOUT, symbol Connector:Test_Point
- U2: renamed from U?; footprint (none) -> sdr-transmitter:ANALOG-LFCSP-VQ-56; symbol ADRF6755 -> sdr-transmitter:ADRF6755
Connections:
- net GND: now also U2.57 (AGND), C19.1, C22.1, C23.1, C24.1, C25.1, C26.1, C27.1, C28.1, C29.1, C30.1, C31.1, C32.1, C33.1, C34.1, C35.1, C36.1, C37.1, C38.1, C39.1, C4.1, C40.1, C41.1, C42.2, C7.1, D2.1 (K), R5.1; no longer U2.EP (AGND)
- net RFOUT: now also C15.1; no longer U2.48 (RFOUT)
- net +5V: now reaches U2.1 (VCC4)
- net +5V: now also U2.11 (VCC1), U2.41 (VCC3), U2.42 (VCC3), U2.55 (VCC2), U2.56 (VCC2), C22.2, C23.2, C24.2, C25.2, C26.2, C27.2, C4.2, C7.2
- net at U2.12 (REGOUT): now also U2.13 (VREG1), U2.14 (VREG2), U2.15 (VREG3), U2.16 (VREG4), U2.25 (LOMON), U2.26 (~LOMON), U2.31 (VREG5), U2.36 (VREG6), C19.2, C29.2, C32.2, C33.2, C34.2, C35.2, C36.2, C37.2, C38.2, C39.2, C40.2, C41.2, C42.1
- net at U2.33 (CCOMP1): now also C28.2
- net at U2.34 (CCOMP2): now also C30.2
- net at U2.35 (CCOMP3): now also C31.2
- net at U2.43 (MUXOUT): now also TP1.1
- net at U2.44 (LDET): now also R6.2
- net at U2.7 (RSET): now also R5.2
- new net: C15.2, U2.48 (RFOUT)
- new net: D2.2 (A), R6.1
Other:
- moved on the sheet: U2
