File: hardware/pa.sch (KiCad schematic (older format))
At the start: 17 parts

Commit message: Update PA matching circuits
Parts:
- removed C? (x4): C, symbol C
- removed C?: CP, symbol CP
- removed C?: 1uF, symbol C
- removed C?: 2.2uF, symbol C
- removed D?: D, symbol D
- removed L?: L, symbol L
- removed RV?: POT_TRIM, symbol POT_TRIM
- removed U?: LP2950-3.3_TO252, TO_SOT_Packages_THT:TO-252-2, symbol LP2950-3.3_TO252
- added C1, C8: 1nF, Capacitors_SMD:C_0603, symbol device:C
- added C10, C5, C?: 100nF, Capacitors_SMD:C_0603, symbol device:C
- added C13: 10nF, Capacitors_SMD:C_0805, symbol device:C
- added C18: 9.1pF, Capacitors_SMD:C_0603, symbol device:C
- added C2: 10pF, Capacitors_SMD:C_0603, symbol device:C
- added C20: 91p, Capacitors_SMD:C_0805, symbol device:C
- added C21, C?: 24pF, Capacitors_SMD:C_0603, symbol device:C
- added C3: 33pF, Capacitors_SMD:C_0603, symbol device:C
- added C6, C?: 100pF, Capacitors_SMD:C_0603, symbol device:C
- added C? (x2): 2.2µF, Capacitors_SMD:C_0603, symbol device:C
- added C?: 10uF, Capacitors_SMD:CP_Elec_10x10.5, symbol device:CP
- added C?: 100n, Capacitors_SMD:C_0603, symbol device:C
- added IM1: PA_Input_Match, sdr-transmitter:PA_Input_Match, symbol sdr-transmitter:PA_Input_Match
- added IM2: PA_Output_Match, sdr-transmitter:PA_Output_Match, symbol sdr-transmitter:PA_Output_Match
- added IM3: Driver_Input_Match, sdr-transmitter:Driver_Input_Match, symbol sdr-transmitter:Driver_Input_Match
- added IM4: Driver_Output_Match, sdr-transmitter:Driver_Output_Match, symbol sdr-transmitter:Driver_Output_Match
- added L1: 47nH, symbol device:L
- added L? (x2): Ferrite_Bead_Small, symbol device:Ferrite_Bead_Small
- added R2: 100, symbol device:R
- added R3: 100, Resistors_SMD:R_1206, symbol device:R
- added R?: 0.05, symbol device:R_Shunt
- added U1: BGA7027, TO_SOT_Packages_SMD:SOT-89-3_Handsoldering, symbol sdr-transmitter:BGA7027
- added U?: AD8217, Housings_SSOP:MSOP-8_3x3mm_Pitch0.65mm, symbol linear:AD8217
- added U?: MCP4726, TO_SOT_Packages_SMD:SOT-23-6, symbol sdr-transmitter:MCP4726
- 1nF1: renamed from C?; footprint (none) -> Capacitors_SMD:C_0603; symbol C -> device:C
- C12: renamed from C?; value C -> 18pF; footprint (none) -> Capacitors_SMD:C_0805; symbol C -> device:C; Digikey (none) -> 490-3606-1-ND; MPN (none) -> GQM2195C2A180JB01D; Mouser (none) -> 81-GQM2195C2A180JB01
- C14: renamed from C?; value C -> 100p; footprint (none) -> Capacitors_SMD:C_0603; symbol C -> device:C
- C17: renamed from C?; value CP -> 330uF; footprint (none) -> Capacitors_SMD:CP_Elec_10x10.5; symbol CP -> device:CP
- L3: renamed from L?; value L -> 33nH; footprint (none) -> sdr-transmitter:1111SQ-33N; symbol L -> device:L; MPN (none) -> 1111SQ-33N
- U4: renamed from U?; footprint (none) -> sdr-transmitter:PLD-1.5W; symbol AFT09MS015N -> sdr-transmitter:AFT09MS015N
Connections:
- net GND: now also C10.2, C18.2, C2.2, C20.2, C21.2, C3.2, C5.2, C6.2, C?.1, C?.2, C?.2, C?.2, C?.2, C?.2, C?.2, U1.2, U?.2 (VSS), U?.4 (GND)
- net RF_IN: now also C1.2
- net VCC: now also R?.1; no longer C14.1, C17.1, L3.1
- net at U4.1: now also IM2.1 (VDD); no longer C12.1
- new net: IM1.1 (In), U4.2
- new net: C12.1, IM1.1 (In)
- new net: 1nF1.2, IM2.1 (VDD)
- new net: C14.1, C17.1, C?.1, L3.1, R?.4
- new net: IM2.1 (VDD), L3.2
- new net: C20.1, IM1.1 (In)
- new net: C18.1, IM2.1 (VDD)
- new net: C21.1, IM2.1 (VDD)
- new net: C2.1, IM3.1 (In)
- new net: C3.1, IM3.1 (In)
- new net: IM4.1 (VDD), U1.1
- new net: IM3.1 (In), U1.3
- new net: C1.1, IM3.1 (In)
- new net: C8.1, IM1.1 (In)
- new net: C8.2, IM4.1 (VDD)
- new net: C5.1, C6.1, C?.1, L1.1, L?.1
- new net: IM4.1 (VDD), L1.2
- new net: C10.1, C?.1, C?.1, L?.1, R2.1
- new net: C13.1, IM2.1 (VDD)
- new net: C?.2, IM2.1 (VDD)
- new net: R?.2, U?.1 (+IN)
- new net: R?.3, U?.8 (-IN)
- new net: L?.2, U?.1 (VOUT)
- new net: IM1.1 (In), R2.2
- new net: IM1.1 (In), R3.2
- new net: C13.2, R3.1
- new net +5V: C?.1, C?.1, L?.2, U?.3 (VDD)
- new net Id: U?.5 (OUT)
- new net SCL: U?.5 (SCL)
- new net SDA: U?.4 (SDA)
- no-connect marks 0 -> 1
Other:
- note removed: "Thermally Coupled\n(see NXP AN1643)"
- moved on the sheet: 1nF1, C12, C14, C17, L3, U4
