File: hardware/sdr-transmitter.kicad_pcb (KiCad board)
At the start: 2 copper layers, 0 parts

Commit message: Update PA matching circuits
Parts:
- added 1nF1: C, Capacitors_SMD:C_0603, F.Cu at (158.2, 144.8)
- added C1: 1nF, Capacitors_SMD:C_0603, F.Cu at (116.6, 111.6)
- added C10: 100n, Capacitors_SMD:C_0603, F.Cu at (110.4, 132.3)
- added C11: 2.2uF, Capacitors_SMD:C_0603, F.Cu at (141.1, 117.3)
- added C12: 18pF, Capacitors_SMD:C_0805, F.Cu at (112.8, 132.0)
- added C13: 10nF, Capacitors_SMD:C_0805, F.Cu at (159.7, 138.9)
- added C14: 100p, Capacitors_SMD:C_0603, F.Cu at (161.5, 125.0)
- added C16: 24pF, Capacitors_SMD:C_0603, F.Cu at (174.8, 137.3)
- added C17: 330uF, Capacitors_SMD:CP_Elec_10x10.5, F.Cu at (164.5, 117.5)
- added C18: 9.1pF, Capacitors_SMD:C_0603, F.Cu at (161.5, 143.1)
- added C19: 100n, Capacitors_SMD:C_0603, F.Cu at (162.0, 86.2)
- added C2: 10pF, Capacitors_SMD:C_0603, F.Cu at (131.0, 103.1)
- added C20: 91p, Capacitors_SMD:C_0805, F.Cu at (137.5, 131.0)
- added C21: 24pF, Capacitors_SMD:C_0603, F.Cu at (174.9, 132.6)
- added C22: 100n, Capacitors_SMD:C_0603, F.Cu at (128.2, 91.7)
- added C23: 10p, Capacitors_SMD:C_0603, F.Cu at (162.0, 91.2)
- added C24: 100n, Capacitors_SMD:C_0603, F.Cu at (111.9, 96.7)
- added C25: 10p, Capacitors_SMD:C_0603, F.Cu at (166.3, 86.2)
- added C26: 100n, Capacitors_SMD:C_0603, F.Cu at (116.2, 91.7)
- added C27: 10p, Capacitors_SMD:C_0603, F.Cu at (170.6, 86.2)
- added C28: 100n, Capacitors_SMD:C_0603, F.Cu at (166.3, 91.2)
- added C29: 10p, Capacitors_SMD:C_0603, F.Cu at (170.6, 91.2)
- added C3: 33pF, Capacitors_SMD:C_0603, F.Cu at (126.9, 108.1)
- added C30: 100n, Capacitors_SMD:C_0603, F.Cu at (111.9, 101.8)
- added C31: 100n, Capacitors_SMD:C_0603, F.Cu at (120.5, 91.7)
- added C32: 100n, Capacitors_SMD:C_0603, F.Cu at (116.2, 96.7)
- added C33: 10p, Capacitors_SMD:C_0603, F.Cu at (120.0, 96.7)
- added C34: 100n, Capacitors_SMD:C_0603, F.Cu at (116.2, 101.8)
- added C35: 10p, Capacitors_SMD:C_0603, F.Cu at (124.4, 91.7)
- added C36: 100n, Capacitors_SMD:C_0603, F.Cu at (111.9, 91.7)
- added C37: 10p, Capacitors_SMD:C_0603, F.Cu at (120.0, 101.8)
- added C38: 100n, Capacitors_SMD:C_0603, F.Cu at (123.9, 96.7)
- added C39: 10p, Capacitors_SMD:C_0603, F.Cu at (127.8, 96.7)
- added C4: 100n, Capacitors_SMD:C_0603, F.Cu at (131.0, 108.1)
- added C40: 100n, Capacitors_SMD:C_0603, F.Cu at (123.9, 101.8)
- added C41: 10p, Capacitors_SMD:C_0603, F.Cu at (132.1, 91.7)
- added C5: 100nF, Capacitors_SMD:C_0603, F.Cu at (122.4, 108.1)
- added C6: 100pF, Capacitors_SMD:C_0603, F.Cu at (126.5, 103.1)
- added C7: 10p, Capacitors_SMD:C_0603, F.Cu at (121.9, 103.1)
- added C8: 1nF, Capacitors_SMD:C_0603, F.Cu at (113.3, 111.6)
- added C9: 1uF, Capacitors_SMD:C_0603, F.Cu at (140.5, 109.5)
- added D2: LED, LEDs:LED_0603, F.Cu at (131.2, 96.5)
- added IM1: PA_Input_Match, sdr-transmitter:PA_Input_Match, F.Cu at (149.4, 138.5)
- added IM2: PA_Output_Match, sdr-transmitter:PA_Output_Match, F.Cu at (156.9, 135.0)
- added IM3: Driver_Input_Match, sdr-transmitter:Driver_Input_Match, F.Cu at (135.3, 145.8)
- added IM4: Driver_Output_Match, sdr-transmitter:Driver_Output_Match, F.Cu at (131.6, 134.1)
- added L3: 33nH, Inductors_SMD:L_1210, F.Cu at (159.6, 130.6)
- added R3: 100, Resistors_SMD:R_1206, F.Cu at (148.8, 139.3)
- added R5: 4k7, Resistors_SMD:R_0603, F.Cu at (127.7, 101.7)
- added R6: 100, Resistors_SMD:R_0603, F.Cu at (135.5, 91.6)
- added U1: BGA7027, TO_SOT_Packages_SMD:SOT-89-3_Handsoldering, F.Cu at (112.4, 100.0)
- added U2: ADRF6755, sdr-transmitter:ANALOG-LFCSP-VQ-56, F.Cu at (154.0, 89.6)
- added U4: AFT09MS015N, sdr-transmitter:PLD-1.5W, F.Cu at (153.8, 135.0)
Other:
- board outline added: 100 x 100 mm
